File: RSHP-MB.kicad_sch (KiCad schematic)
At the start: 23 parts, among them J1 Conn_02x20_Odd_Even, J2 Conn_02x02_Odd_Even, J3 Conn_02x02_Odd_Even, J4 Conn_02x04_Odd_Even

Commit message: Changed mount holes to M4 diameter. Generated CAM files.
Parts:
- H12, H13, H14, H15: footprint MountingHole:MountingHole_5.3mm_M5_Pad -> MountingHole:MountingHole_4.3mm_M4_Pad
Changed lines of the file:
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@@
   (title_block
     (title "RSHP-MB-0010")
-    (date "2022-05-22")
+    (date "2022-05-25")
     (rev "1.0")
     (company "(c) Andriy Golovnya http://redscorp.net")
@@
       (effects (font (size 1.27 1.27)) (justify left))
     )
-    (property "Footprint" "MountingHole:MountingHole_5.3mm_M5_Pad" (id 2) (at 140.97 120.65 0)
+    (property "Footprint" "MountingHole:MountingHole_4.3mm_M4_Pad" (id 2) (at 140.97 120.65 0)
       (effects (font (size 1.27 1.27)) hide)
     )
@@
       (effects (font (size 1.27 1.27)) (justify left))
     )
-    (property "Footprint" "MountingHole:MountingHole_5.3mm_M5_Pad" (id 2) (at 140.97 125.73 0)
+    (property "Footprint" "MountingHole:MountingHole_4.3mm_M4_Pad" (id 2) (at 140.97 125.73 0)
       (effects (font (size 1.27 1.27)) hide)
     )
@@
       (effects (font (size 1.27 1.27)) (justify left))
     )
-    (property "Footprint" "MountingHole:MountingHole_5.3mm_M5_Pad" (id 2) (at 140.97 135.89 0)
+    (property "Footprint" "MountingHole:MountingHole_4.3mm_M4_Pad" (id 2) (at 140.97 135.89 0)
       (effects (font (size 1.27 1.27)) hide)
     )
@@
       (effects (font (size 1.27 1.27)) (justify left))
     )
-    (property "Footprint" "MountingHole:MountingHole_5.3mm_M5_Pad" (id 2) (at 140.97 130.81 0)
+    (property "Footprint" "MountingHole:MountingHole_4.3mm_M4_Pad" (id 2) (at 140.97 130.81 0)
       (effects (font (size 1.27 1.27)) hide)
     )
@@
     )
     (path "/3efb45eb-a1cc-4300-85c8-c7f83adc9f7d"
-      (reference "H12") (unit 1) (value "MountingHole") (footprint "MountingHole:MountingHole_5.3mm_M5_Pad")
+      (reference "H12") (unit 1) (value "MountingHole") (footprint "MountingHole:MountingHole_4.3mm_M4_Pad")
     )
     (path "/578f9548-2849-49c1-88c1-08aad6adf0a0"
-      (reference "H13") (unit 1) (value "MountingHole") (footprint "MountingHole:MountingHole_5.3mm_M5_Pad")
+      (reference "H13") (unit 1) (value "MountingHole") (footprint "MountingHole:MountingHole_4.3mm_M4_Pad")
     )
     (path "/f827d236-9ee6-43a7-a617-285ccd803ee7"
-      (reference "H14") (unit 1) (value "MountingHole") (footprint "MountingHole:MountingHole_5.3mm_M5_Pad")
+      (reference "H14") (unit 1) (value "MountingHole") (footprint "MountingHole:MountingHole_4.3mm_M4_Pad")
     )
     (path "/c4ad4b68-2119-41a7-aefb-1c09d3373e77"
-      (reference "H15") (unit 1) (value "MountingHole") (footprint "MountingHole:MountingHole_5.3mm_M5_Pad")
+      (reference "H15") (unit 1) (value "MountingHole") (footprint "MountingHole:MountingHole_4.3mm_M4_Pad")
     )
     (path "/1747e309-d2e2-4752-b7fc-5a3f12028340"
